File: hardware/base-plane/base-plane.kicad_pcb (KiCad board)
At the start: 6 copper layers, 124.5 x 50.8 mm, 155 parts, among them J1 Conn_01x02_Female, J10 Conn_01x02, J11 Conn_01x05, J12 Conn_02x10_Odd_Even, J13 FH12-24S-0.5SH(55), J2 USB_Connectors_USB_3.0_MICRO-B, J3 USB3_A, J4 Conn_01x06, J5 Conn_01x06, J6 Conn_01x06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

Commit message: kleinere Anpassungen
Routing:
- net Net-(R20-Pad2): track 23.8 -> 22.1 mm
