File: hardware/base-plane/hub.sch (KiCad schematic (older format))
At the start: 31 parts, among them U3 TUSB8041ARGCR, Y1 24MHz

Commit message: kleinere Anpassungen
Parts:
- removed R8: 90.9k 1%, Resistor_SMD:R_0603_1608Metric, symbol Device:R
- removed R9: 10k 1%, Resistor_SMD:R_0603_1608Metric, symbol Device:R
- R12: value 40k -> 4.7k
Connections:
- net USB_VBUS: now also U3.48 (USB_VBUS)
Changed lines of the file:
@@
 P 10500 2650
 F 0 "R12" H 10570 2696 50  0000 L CNN
-F 1 "40k" H 10570 2605 50  0000 L CNN
+F 1 "4.7k" H 10570 2605 50  0000 L CNN
 F 2 "Resistor_SMD:R_0603_1608Metric" V 10430 2650 50  0001 C CNN
 F 3 "~" H 10500 2650 50  0001 C CNN
@@
 Text GLabel 10300 4000 0    50   Input ~ 0
 FULLPWRMGMTZ
-$Comp
-L Device:R R9
-U 1 1 60C47D8A
-P 2400 3300
-F 0 "R9" H 2470 3346 50  0000 L CNN
-F 1 "10k 1%" H 2470 3255 50  0000 L CNN
-F 2 "Resistor_SMD:R_0603_1608Metric" V 2330 3300 50  0001 C CNN
-F 3 "~" H 2400 3300 50  0001 C CNN
-	1    2400 3300
-	1    0    0    -1
-$EndComp
-$Comp
-L Device:R R8
-U 1 1 60C48806
-P 2200 3050
-F 0 "R8" V 1993 3050 50  0000 C CNN
-F 1 "90.9k 1%" V 2084 3050 50  0000 C CNN
-F 2 "Resistor_SMD:R_0603_1608Metric" V 2130 3050 50  0001 C CNN
-F 3 "~" H 2200 3050 50  0001 C CNN
-	1    2200 3050
-	0    1    1    0
-$EndComp
-Wire Wire Line
-	2350 3050 2400 3050
-Wire Wire Line
-	2400 3150 2400 3050
-Connection ~ 2400 3050
-Wire Wire Line
-	2400 3050 3850 3050
-Wire Wire Line
-	2050 3050 1850 3050
-$Comp
-L power:GND #PWR034
-U 1 1 60C58F2D
-P 2400 3500
-F 0 "#PWR034" H 2400 3250 50  0001 C CNN
-F 1 "GND" H 2405 3327 50  0000 C CNN
-F 2 "" H 2400 3500 50  0001 C CNN
-F 3 "" H 2400 3500 50  0001 C CNN
-	1    2400 3500
-	1    0    0    -1
-$EndComp
-Wire Wire Line
-	2400 3500 2400 3450
 Text Notes 9950 2200 0    50   ~ 0
 SMBus Mode Selected???
@@
 Wire Wire Line
 	3450 5650 3850 5650
+Wire Wire Line
+	1850 3050 3850 3050
 Wire Bus Line
 	8400 4500 8400 5350
