File: hardware/port-plane/port-plane/input.sch (KiCad schematic (older format))
At the start: 22 parts, among them J1 Conn_01x06, J2 Conn_01x02_Female, J3 USB_Connectors_USB_3.0_MICRO-B

Commit message: kleinere Anpassungen
Parts:
- J2: footprint Connector_Molex:Molex_Mini-Fit_Jr_5566-02A_2x01_P4.20mm_Vertical -> Connector_Molex:Molex_Mini-Fit_Jr_5569-02A2_2x01_P4.20mm_Horizontal
- gave numbers to parts that had none: 2
Changed lines of the file:
@@
 F 0 "J2" H 5392 1975 50  0000 C CNN
 F 1 "Conn_01x02_Female" H 5392 2066 50  0001 C CNN
-F 2 "Connector_Molex:Molex_Mini-Fit_Jr_5566-02A_2x01_P4.20mm_Vertical" H 5500 2300 50  0001 C CNN
+F 2 "Connector_Molex:Molex_Mini-Fit_Jr_5569-02A2_2x01_P4.20mm_Horizontal" H 5500 2300 50  0001 C CNN
 F 3 "~" H 5500 2300 50  0001 C CNN
 	1    5500 2300
@@
 Connection ~ 3900 2350
 $Comp
-L Device:R R?
+L Device:R R31
 U 1 1 60423E79
 P 3600 4350
-F 0 "R?" H 3670 4396 50  0000 L CNN
+F 0 "R31" H 3670 4396 50  0000 L CNN
 F 1 "R" H 3670 4305 50  0000 L CNN
 F 2 "" V 3530 4350 50  0001 C CNN
@@
 $EndComp
 $Comp
-L Device:R R?
+L Device:R R32
 U 1 1 60424D85
 P 3950 4350
-F 0 "R?" H 4020 4396 50  0000 L CNN
+F 0 "R32" H 4020 4396 50  0000 L CNN
 F 1 "R" H 4020 4305 50  0000 L CNN
 F 2 "" V 3880 4350 50  0001 C CNN
@@
 	3950 4750 4100 4750
 $Comp
-L power:+3.3V #PWR?
+L power:+3.3V #PWR0101
 U 1 1 6042D387
 P 3800 3900
-F 0 "#PWR?" H 3800 3750 50  0001 C CNN
+F 0 "#PWR0101" H 3800 3750 50  0001 C CNN
 F 1 "+3.3V" H 3815 4073 50  0000 C CNN
 F 2 "" H 3800 3900 50  0001 C CNN
