File: hardware/port-plane/port-plane/user_interface.sch (KiCad schematic (older format))
At the start: 25 parts, among them SW1 TA-633N-V-T_R, SW2 TA-633N-V-T_R, SW3 TA-633N-V-T_R, SW4 TA-633N-V-T_R, U7 LP5012PWR, U8 MAX7323AEE+, U9 LP5012PWR

Commit message: kleinere Anpassungen
Parts:
- removed D1, D2, D3, D4, D5, D6, D7, D8: MSL0601RGB, leds_and_switches:MSL0601RGB, symbol Device:LED_BGRA
- added D1, D2, D3, D4, D5, D6, D7, D8: LED_RGB, leds_and_switches:KRTB_AELPS1.32, symbol Device:LED_RGB
Connections:
- net +3V3: now also D1.4 (BA), D1.5 (GA), D1.6 (RA), D2.4 (BA), D2.5 (GA), D2.6 (RA), D3.4 (BA), D3.5 (GA), D3.6 (RA), D4.4 (BA), D4.5 (GA), D4.6 (RA), D5.4 (BA), D5.5 (GA), D5.6 (RA), D6.4 (BA), D6.5 (GA), D6.6 (RA), D7.4 (BA), D7.5 (GA), D7.6 (RA), D8.4 (BA), D8.5 (GA), D8.6 (RA)
- net at U7.14 (Out2): now also D1.3 (BK)
- net at U7.13 (Out1): now also D1.2 (GK)
- net at U7.12 (Out0): now also D1.1 (RK)
- net at U7.17 (Out5): now also D2.3 (BK)
- net at U7.16 (Out4): now also D2.2 (GK)
- net at U7.15 (Out3): now also D2.1 (RK)
- net at U7.21 (Out8): now also D3.3 (BK)
- net at U7.20 (Out7): now also D3.2 (GK)
- net at U7.19 (Out6): now also D3.1 (RK)
- net at U7.24 (Out11): now also D4.3 (BK)
- net at U7.23 (Out10): now also D4.2 (GK)
- net at U7.22 (Out9): now also D4.1 (RK)
- net at U9.14 (Out2): now also D5.3 (BK)
- net at U9.13 (Out1): now also D5.2 (GK)
- net at U9.12 (Out0): now also D5.1 (RK)
- net at U9.17 (Out5): now also D6.3 (BK)
- net at U9.16 (Out4): now also D6.2 (GK)
- net at U9.15 (Out3): now also D6.1 (RK)
- net at U9.21 (Out8): now also D7.3 (BK)
- net at U9.20 (Out7): now also D7.2 (GK)
- net at U9.19 (Out6): now also D7.1 (RK)
- net at U9.24 (Out11): now also D8.3 (BK)
- net at U9.23 (Out10): now also D8.2 (GK)
- net at U9.22 (Out9): now also D8.1 (RK)
Changed lines of the file:
@@
 	4150 6050 3550 6050
-$Comp
-L Device:LED_BGRA D1
-U 1 1 60518DEF
-P 4100 1500
-F 0 "D1" H 4100 1997 50  0000 C CNN
-F 1 "MSL0601RGB" H 4100 1906 50  0000 C CNN
-F 2 "leds_and_switches:MSL0601RGB" H 4100 1450 50  0001 C CNN
-F 3 "https://www.mouser.de/datasheet/2/348/msl0601rgb-e-1874495.pdf~" H 4100 1450 50  0001 C CNN
-	1    4100 1500
-	1    0    0    -1
-$EndComp
-$Comp
-L Device:LED_BGRA D2
-U 1 1 60518DF5
-P 4100 2400
-F 0 "D2" H 4100 2897 50  0000 C CNN
-F 1 "MSL0601RGB" H 4100 2806 50  0000 C CNN
-F 2 "leds_and_switches:MSL0601RGB" H 4100 2350 50  0001 C CNN
-F 3 "~" H 4100 2350 50  0001 C CNN
-	1    4100 2400
-	1    0    0    -1
-$EndComp
-$Comp
-L Device:LED_BGRA D3
-U 1 1 60518DFB
-P 4100 3300
-F 0 "D3" H 4100 3797 50  0000 C CNN
-F 1 "MSL0601RGB" H 4100 3706 50  0000 C CNN
-F 2 "leds_and_switches:MSL0601RGB" H 4100 3250 50  0001 C CNN
-F 3 "~" H 4100 3250 50  0001 C CNN
-	1    4100 3300
-	1    0    0    -1
-$EndComp
-$Comp
-L Device:LED_BGRA D4
-U 1 1 60518E01
-P 4100 4200
-F 0 "D4" H 4100 4697 50  0000 C CNN
-F 1 "MSL0601RGB" H 4100 4606 50  0000 C CNN
-F 2 "leds_and_switches:MSL0601RGB" H 4100 4150 50  0001 C CNN
-F 3 "~" H 4100 4150 50  0001 C CNN
-	1    4100 4200
-	1    0    0    -1
-$EndComp
 $Comp
 L io:LP5012PWR U7
@@
 $EndComp
 Wire Wire Line
-	4650 1150 4650 1500
-Wire Wire Line
-	4650 4200 4300 4200
-Wire Wire Line
-	4650 3300 4300 3300
-Connection ~ 4650 3300
-Wire Wire Line
-	4650 3300 4650 4200
-Wire Wire Line
-	4650 2400 4300 2400
-Connection ~ 4650 2400
-Wire Wire Line
-	4650 2400 4650 3300
-Wire Wire Line
-	4650 1500 4300 1500
-Connection ~ 4650 1500
-Wire Wire Line
-	4650 1500 4650 2400
-Wire Wire Line
 	3900 1300 3150 1300
 Wire Wire Line
@@
 Addr: 0x14\nBroadc.: 0x0C
 $Comp
-L Device:LED_BGRA D5
-U 1 1 6057A6C2
-P 9450 1500
-F 0 "D5" H 9450 1997 50  0000 C CNN
-F 1 "MSL0601RGB" H 9450 1906 50  0000 C CNN
-F 2 "leds_and_switches:MSL0601RGB" H 9450 1450 50  0001 C CNN
-F 3 "https://www.mouser.de/datasheet/2/348/msl0601rgb-e-1874495.pdf~" H 9450 1450 50  0001 C CNN
-	1    9450 1500
-	1    0    0    -1
-$EndComp
-$Comp
-L Device:LED_BGRA D6
-U 1 1 6057A6C8
-P 9450 2400
-F 0 "D6" H 9450 2897 50  0000 C CNN
-F 1 "MSL0601RGB" H 9450 2806 50  0000 C CNN
-F 2 "leds_and_switches:MSL0601RGB" H 9450 2350 50  0001 C CNN
-F 3 "~" H 9450 2350 50  0001 C CNN
-	1    9450 2400
-	1    0    0    -1
-$EndComp
-$Comp
-L Device:LED_BGRA D7
-U 1 1 6057A6CE
-P 9450 3300
-F 0 "D7" H 9450 3797 50  0000 C CNN
-F 1 "MSL0601RGB" H 9450 3706 50  0000 C CNN
-F 2 "leds_and_switches:MSL0601RGB" H 9450 3250 50  0001 C CNN
-F 3 "~" H 9450 3250 50  0001 C CNN
-	1    9450 3300
-	1    0    0    -1
-$EndComp
-$Comp
-L Device:LED_BGRA D8
-U 1 1 6057A6D4
-P 9450 4200
-F 0 "D8" H 9450 4697 50  0000 C CNN
-F 1 "MSL0601RGB" H 9450 4606 50  0000 C CNN
-F 2 "leds_and_switches:MSL0601RGB" H 9450 4150 50  0001 C CNN
-F 3 "~" H 9450 4150 50  0001 C CNN
-	1    9450 4200
-	1    0    0    -1
-$EndComp
-$Comp
 L io:LP5012PWR U9
 U 1 1 6057A6DA
@@
 $EndComp
 Wire Wire Line
-	10000 1150 10000 1500
+	10000 1150 10000 1300
 Wire Wire Line
 	10000 4200 9650 4200
@@
 Connection ~ 10000 3300
 Wire Wire Line
-	10000 3300 10000 4200
+	10000 3300 10000 3500
 Wire Wire Line
 	10000 2400 9650 2400
 Connection ~ 10000 2400
 Wire Wire Line
-	10000 2400 10000 3300
+	10000 2400 10000 2600
 Wire Wire Line
 	10000 1500 9650 1500
 Connection ~ 10000 1500
 Wire Wire Line
-	10000 1500 10000 2400
+	10000 1500 10000 1700
 Wire Wire Line
 	9250 1300 8500 1300
@@
 Wire Wire Line
 	4300 6300 5200 6300
+$Comp
+L Device:LED_RGB D1
+U 1 1 605C0F90
+P 4100 1500
+F 0 "D1" H 4100 1997 50  0000 C CNN
+F 1 "LED_RGB" H 4100 1906 50  0000 C CNN
+F 2 "leds_and_switches:KRTB_AELPS1.32" H 4100 1450 50  0001 C CNN
+F 3 "~" H 4100 1450 50  0001 C CNN
+	1    4100 1500
+	1    0    0    -1
+$EndComp
+$Comp
+L Device:LED_RGB D2
+U 1 1 605C69A0
+P 4100 2400
+F 0 "D2" H 4100 2897 50  0000 C CNN
+F 1 "LED_RGB" H 4100 2806 50  0000 C CNN
+F 2 "leds_and_switches:KRTB_AELPS1.32" H 4100 2350 50  0001 C CNN
+F 3 "~" H 4100 2350 50  0001 C CNN
+	1    4100 2400
+	1    0    0    -1
+$EndComp
+$Comp
+L Device:LED_RGB D3
+U 1 1 605C86C1
+P 4100 3300
+F 0 "D3" H 4100 3797 50  0000 C CNN
+F 1 "LED_RGB" H 4100 3706 50  0000 C CNN
+F 2 "leds_and_switches:KRTB_AELPS1.32" H 4100 3250 50  0001 C CNN
+F 3 "~" H 4100 3250 50  0001 C CNN
+	1    4100 3300
+	1    0    0    -1
+$EndComp
+$Comp
+L Device:LED_RGB D4
+U 1 1 605C9FCD
+P 4100 4200
+F 0 "D4" H 4100 4697 50  0000 C CNN
+F 1 "LED_RGB" H 4100 4606 50  0000 C CNN
+F 2 "leds_and_switches:KRTB_AELPS1.32" H 4100 4150 50  0001 C CNN
+F 3 "~" H 4100 4150 50  0001 C CNN
+	1    4100 4200
+	1    0    0    -1
+$EndComp
+Wire Wire Line
+	4650 4400 4300 4400
+Wire Wire Line
+	4650 1150 4650 1300
+Wire Wire Line
+	4300 4200 4650 4200
+Connection ~ 4650 4200
+Wire Wire Line
+	4650 4200 4650 4400
+Wire Wire Line
+	4300 4000 4650 4000
+Connection ~ 4650 4000
+Wire Wire Line
+	4650 4000 4650 4200
+Wire Wire Line
+	4300 3500 4650 3500
+Connection ~ 4650 3500
+Wire Wire Line
+	4650 3500 4650 4000
+Wire Wire Line
+	4300 3300 4650 3300
+Connection ~ 4650 3300
+Wire Wire Line
+	4650 3300 4650 3500
+Connection ~ 4650 3100
+Wire Wire Line
+	4650 3100 4650 3300
+Wire Wire Line
+	4300 3100 4650 3100
+Wire Wire Line
+	4300 2200 4650 2200
+Connection ~ 4650 2200
+Wire Wire Line
+	4650 2200 4650 2400
+Wire Wire Line
+	4300 2400 4650 2400
+Connection ~ 4650 2400
+Wire Wire Line
+	4650 2400 4650 2600
+Wire Wire Line
+	4300 2600 4650 2600
+Connection ~ 4650 2600
+Wire Wire Line
+	4650 2600 4650 3100
+Wire Wire Line
+	4300 1300 4650 1300
+Connection ~ 4650 1300
+Wire Wire Line
+	4650 1300 4650 1500
+Wire Wire Line
+	4300 1500 4650 1500
+Connection ~ 4650 1500
+Wire Wire Line
+	4650 1500 4650 1700
+Wire Wire Line
+	4300 1700 4650 1700
+Connection ~ 4650 1700
+Wire Wire Line
+	4650 1700 4650 2200
+$Comp
+L Device:LED_RGB D5
+U 1 1 6063FF74
+P 9450 1500
+F 0 "D5" H 9450 1997 50  0000 C CNN
+F 1 "LED_RGB" H 9450 1906 50  0000 C CNN
+F 2 "leds_and_switches:KRTB_AELPS1.32" H 9450 1450 50  0001 C CNN
+F 3 "~" H 9450 1450 50  0001 C CNN
+	1    9450 1500
+	1    0    0    -1
+$EndComp
+$Comp
+L Device:LED_RGB D6
+U 1 1 60641010
+P 9450 2400
+F 0 "D6" H 9450 2897 50  0000 C CNN
+F 1 "LED_RGB" H 9450 2806 50  0000 C CNN
+F 2 "leds_and_switches:KRTB_AELPS1.32" H 9450 2350 50  0001 C CNN
+F 3 "~" H 9450 2350 50  0001 C CNN
+	1    9450 2400
+	1    0    0    -1
+$EndComp
+$Comp
+L Device:LED_RGB D7
+U 1 1 6064202A
+P 9450 3300
+F 0 "D7" H 9450 3797 50  0000 C CNN
+F 1 "LED_RGB" H 9450 3706 50  0000 C CNN
+F 2 "leds_and_switches:KRTB_AELPS1.32" H 9450 3250 50  0001 C CNN
+F 3 "~" H 9450 3250 50  0001 C CNN
+	1    9450 3300
+	1    0    0    -1
+$EndComp
+$Comp
+L Device:LED_RGB D8
+U 1 1 60643111
+P 9450 4200
+F 0 "D8" H 9450 4697 50  0000 C CNN
+F 1 "LED_RGB" H 9450 4606 50  0000 C CNN
+F 2 "leds_and_switches:KRTB_AELPS1.32" H 9450 4150 50  0001 C CNN
+F 3 "~" H 9450 4150 50  0001 C CNN
+	1    9450 4200
+	1    0    0    -1
+$EndComp
+Wire Wire Line
+	9650 4400 10000 4400
+Wire Wire Line
+	10000 4400 10000 4200
+Connection ~ 10000 4200
+Wire Wire Line
+	9650 4000 10000 4000
+Connection ~ 10000 4000
+Wire Wire Line
+	10000 4000 10000 4200
+Wire Wire Line
+	9650 3500 10000 3500
+Connection ~ 10000 3500
+Wire Wire Line
+	10000 3500 10000 4000
+Wire Wire Line
+	9650 3100 10000 3100
+Connection ~ 10000 3100
+Wire Wire Line
+	10000 3100 10000 3300
+Wire Wire Line
+	9650 2600 10000 2600
+Connection ~ 10000 2600
+Wire Wire Line
+	10000 2600 10000 3100
+Wire Wire Line
+	9650 2200 10000 2200
+Connection ~ 10000 2200
+Wire Wire Line
+	10000 2200 10000 2400
+Wire Wire Line
+	9650 1700 10000 1700
+Connection ~ 10000 1700
+Wire Wire Line
+	10000 1700 10000 2200
+Wire Wire Line
+	9650 1300 10000 1300
+Connection ~ 10000 1300
+Wire Wire Line
+	10000 1300 10000 1500
 $EndSCHEMATC
